Commit message: commit.

File: gap_rl/assets/descriptions/indy7/indy_robotiq85_old.urdf (robot description, URDF)
Before this commit: robot indy7_robotiq85_old, 26 links, 22 joints
Joints:
- added joint robotiq_2f_85_left_pad_joint: type fixed, parent left_inner_finger_pad, child robotiq_85_left_finger_tip_link, origin xyz=-0.025 -0.005 0 rpy=0 0 0, axis 0 0 1
- added joint robotiq_2f_85_right_pad_joint: type fixed, parent right_inner_finger_pad, child robotiq_85_right_finger_tip_link, origin xyz=-0.025 -0.005 0 rpy=0 0 0, axis 0 0 1
- added joint robotiq_85_left_finger_joint: type fixed, parent robotiq_85_left_knuckle_link, child robotiq_85_left_finger_link, origin xyz=-0.00408552455 -0.03148604435 0.0 rpy=0 0 0, axis 0 0 1
